Commit message: Removed robot config from common library, and made ik function independent

File: quadruped_ws/src/my_bot_description/urdf/my_robot.urdf (robot description, URDF)
Before this commit: robot transformx_pleasework_Icantdothisonemoretime, 17 links, 16 joints
Links:
- removed link femur 1
- removed link femur 2
- removed link femur 3
- removed link femur 4
- removed link shoulder 1
- removed link shoulder 2
- removed link shoulder 3
- removed link shoulder 4
- removed link wheel 1
- removed link wheel 2
- removed link wheel 3
- removed link wheel 4
- added link femur_1, mass 0.0189108850293239; collision mesh filename=package://my_bot_description/meshes/femur 1.STL; visual mesh filename=package://my_bot_description/meshes/femur 1.STL
- added link femur_2, mass 0.0189108850293239; collision mesh filename=package://my_bot_description/meshes/femur 2.STL; visual mesh filename=package://my_bot_description/meshes/femur 2.STL
- added link femur_3, mass 0.0189108850293239; collision mesh filename=package://my_bot_description/meshes/femur 3.STL; visual mesh filename=package://my_bot_description/meshes/femur 3.STL
- added link femur_4, mass 0.0189108850293239; collision mesh filename=package://my_bot_description/meshes/femur 4.STL; visual mesh filename=package://my_bot_description/meshes/femur 4.STL
- added link shoulder_1, mass 0.0508037942000163; collision mesh filename=package://my_bot_description/meshes/shoulder 1.STL; visual mesh filename=package://my_bot_description/meshes/shoulder 1.STL
- added link shoulder_2, mass 0.0508037942979783; collision mesh filename=package://my_bot_description/meshes/shoulder 2.STL; visual mesh filename=package://my_bot_description/meshes/shoulder 2.STL
- added link shoulder_3, mass 0.0508037978102054; collision mesh filename=package://my_bot_description/meshes/shoulder 3.STL; visual mesh filename=package://my_bot_description/meshes/shoulder 3.STL
- added link shoulder_4, mass 0.050803797524623; collision mesh filename=package://my_bot_description/meshes/shoulder 4.STL; visual mesh filename=package://my_bot_description/meshes/shoulder 4.STL
- added link wheel_1, mass 0.0307487077587976; collision mesh filename=package://my_bot_description/meshes/wheel 1.STL; visual mesh filename=package://my_bot_description/meshes/wheel 1.STL
- added link wheel_2, mass 0.0307487077587974; collision mesh filename=package://my_bot_description/meshes/wheel 2.STL; visual mesh filename=package://my_bot_description/meshes/wheel 2.STL
- added link wheel_3, mass 0.0307487077587975; collision mesh filename=package://my_bot_description/meshes/wheel 3.STL; visual mesh filename=package://my_bot_description/meshes/wheel 3.STL
- added link wheel_4, mass 0.0307487077587974; collision mesh filename=package://my_bot_description/meshes/wheel 4.STL; visual mesh filename=package://my_bot_description/meshes/wheel 4.STL
